Commit message: fix: fix link_left_shoulder_yaw rpy manually

File: phc/data/assets/robot/zhiyuan_x1/urdf/x1.urdf (robot description, URDF)
Before this commit: robot zhiyuan scene, 31 links, 29 joints
Joints:
- joint left_shoulder_yaw_joint: origin xyz=0.0 0.1252 -0.0313 rpy=0.0 1.5707963267948966 0.0 -> xyz=0.0 0.1252 -0.0313 rpy=1.5707997741256383 1.5707963267948966 0.0

File: phc/data/assets/robot/zhiyuan_x1/urdf/x1_ros.urdf (robot description, URDF)
Before this commit: robot zhiyuan scene, 31 links, 29 joints
Joints:
- joint left_shoulder_yaw_joint: origin xyz=0.0 0.1252 -0.0313 rpy=0.0 1.5707963267948966 0.0 -> xyz=0.0 0.1252 -0.0313 rpy=1.5707997741256383 1.5707963267948966 0.0

Commit message: fix: adjust urdf ref to urdf_rviz_joint

File: phc/data/assets/robot/zhiyuan_x1/urdf/x1.urdf (robot description, URDF)
Before this commit: robot zhiyuan scene, 31 links, 29 joints
Joints:
- added joint base_to_x1_body_joint: type fixed, parent base_link, child x1-body, origin xyz=0 0 0 rpy=0 0 0

File: phc/data/assets/robot/zhiyuan_x1/urdf/x1_ros.urdf (robot description, URDF)
Before this commit: robot zhiyuan scene, 31 links, 29 joints
Links:
- link link_left_ankle_pitch: geometry collision mesh filename=package://x1_urdf/robot/x1_29dof/meshes/left_ankle_pitch.STL; visual mesh filename=package://x1_urdf/robot/x1_29dof/meshes/left_ankle_pitch.STL
- link link_left_ankle_roll: geometry collision mesh filename=package://x1_urdf/robot/x1_29dof/meshes/left_ankle_roll.STL; collision sphere radius=0.002
- link link_left_elbow_pitch: geometry collision mesh filename=package://x1_urdf/robot/x1_29dof/meshes/left_elbow_pitch.STL; visual mesh filename=package://x1_urdf/robot/x1_29dof/meshes/left_elbow_pitch.STL
- link link_left_elbow_yaw: geometry collision mesh filename=package://x1_urdf/robot/x1_29dof/meshes/left_elbow_yaw.STL; visual mesh filename=package://x1_urdf/robot/x1_29dof/meshes/left_elbow_yaw.STL
- link link_left_hip_pitch: geometry collision mesh filename=package://x1_urdf/robot/x1_29dof/meshes/left_hip_pitch.STL; visual mesh filename=package://x1_urdf/robot/x1_29dof/meshes/left_hip_pitch.STL
- link link_left_hip_roll: geometry collision mesh filename=package://x1_urdf/robot/x1_29dof/meshes/left_hip_roll.STL; visual mesh filename=package://x1_urdf/robot/x1_29dof/meshes/left_hip_roll.STL
- link link_left_hip_yaw: geometry collision mesh filename=package://x1_urdf/robot/x1_29dof/meshes/left_hip_yaw.STL; visual mesh filename=package://x1_urdf/robot/x1_29dof/meshes/left_hip_yaw.STL
- link link_left_shoulder_pitch: geometry collision mesh filename=package://x1_urdf/robot/x1_29dof/meshes/left_shoulder_pitch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; visual mesh filename=package://x1_urdf/robot/x1_29dof/meshes/left_shoulder_pitch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
- link link_left_shoulder_roll: geometry collision mesh filename=package://x1_urdf/robot/x1_29dof/meshes/left_shoulder_roll.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; visual mesh filename=package://x1_urdf/robot/x1_29dof/meshes/left_shoulder_roll.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
- link link_left_shoulder_yaw: geometry collision mesh filename=package://x1_urdf/robot/x1_29dof/meshes/left_shoulder_yaw.S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; visual mesh filename=package://x1_urdf/robot/x1_29dof/meshes/left_shoulder_yaw.S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
- link link_left_wrist_pitch: geometry collision mesh filename=package://x1_urdf/robot/x1_29dof/meshes/left_wrist_pitch.STL; visual mesh filename=package://x1_urdf/robot/x1_29dof/meshes/left_wrist_pitch.STL
- link link_left_wrist_roll: geometry collision mesh filename=package://x1_urdf/robot/x1_29dof/meshes/left_wrist_roll.STL; visual mesh filename=package://x1_urdf/robot/x1_29dof/meshes/left_wrist_roll.STL
- link link_lleft_knee_pitch: geometry collision mesh filename=package://x1_urdf/robot/x1_29dof/meshes/left_knee_pitch.STL; visual mesh filename=package://x1_urdf/robot/x1_29dof/meshes/left_knee_pitch.STL
- link link_lumbar_pitch: geometry collision mesh filename=package://x1_urdf/robot/x1_29dof/meshes/lumbar_pitch.STL; collision mesh filename=package://x1_urdf/robot/x1_29dof/meshes/lumbar_pitch.STL
- link link_lumbar_roll: geometry collision mesh filename=package://x1_urdf/robot/x1_29dof/meshes/lumbar_roll.STL; visual mesh filename=package://x1_urdf/robot/x1_29dof/meshes/lumbar_roll.STL
- link link_lumbar_yaw: geometry collision mesh filename=package://x1_urdf/robot/x1_29dof/meshes/lumbar_yaw.STL; visual mesh filename=package://x1_urdf/robot/x1_29dof/meshes/lumbar_yaw.STL
- link link_right_ankle_pitch: geometry collision mesh filename=package://x1_urdf/robot/x1_29dof/meshes/right_ankle_pitch.S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; visual mesh filename=package://x1_urdf/robot/x1_29dof/meshes/right_ankle_pitch.S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
- link link_right_ankle_roll: geometry collision mesh filename=package://x1_urdf/robot/x1_29dof/meshes/right_ankle_roll.STL; collision sphere radius=0.002
- link link_right_elbow_pitch: geometry collision mesh filename=package://x1_urdf/robot/x1_29dof/meshes/right_elbow_pitch.S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; visual mesh filename=package://x1_urdf/robot/x1_29dof/meshes/right_elbow_pitch.S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
- link link_right_elbow_yaw: geometry collision mesh filename=package://x1_urdf/robot/x1_29dof/meshes/right_elbow_yaw.STL; visual mesh filename=package://x1_urdf/robot/x1_29dof/meshes/right_elbow_yaw.STL
- link link_right_hip_pitch: geometry collision mesh filename=package://x1_urdf/robot/x1_29dof/meshes/right_hip_pitch.STL; visual mesh filename=package://x1_urdf/robot/x1_29dof/meshes/right_hip_pitch.STL
- link link_right_hip_roll: geometry collision mesh filename=package://x1_urdf/robot/x1_29dof/meshes/right_hip_roll.STL; visual mesh filename=package://x1_urdf/robot/x1_29dof/meshes/right_hip_roll.STL
- link link_right_hip_yaw: geometry collision mesh filename=package://x1_urdf/robot/x1_29dof/meshes/right_hip_yaw.STL; visual mesh filename=package://x1_urdf/robot/x1_29dof/meshes/right_hip_yaw.STL
- link link_right_knee_pitch: geometry collision mesh filename=package://x1_urdf/robot/x1_29dof/meshes/right_knee_pitch.STL; visual mesh filename=package://x1_urdf/robot/x1_29dof/meshes/right_knee_pitch.STL
- link link_right_shoulder_pitch: geometry collision mesh filename=package://x1_urdf/robot/x1_29dof/meshes/right_shoulder_pitc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; visual mesh filename=package://x1_urdf/robot/x1_29dof/meshes/right_shoulder_pitc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
- link link_right_shoulder_roll: geometry collision mesh filename=package://x1_urdf/robot/x1_29dof/meshes/right_shoulder_roll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; visual mesh filename=package://x1_urdf/robot/x1_29dof/meshes/right_shoulder_roll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
- link link_right_shoulder_yaw: geometry collision mesh filename=package://x1_urdf/robot/x1_29dof/meshes/right_shoulder_yaw.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; visual mesh filename=package://x1_urdf/robot/x1_29dof/meshes/right_shoulder_yaw.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
- link link_right_wrist_pitch: geometry collision mesh filename=package://x1_urdf/robot/x1_29dof/meshes/right_wrist_pitch.S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; visual mesh filename=package://x1_urdf/robot/x1_29dof/meshes/right_wrist_pitch.S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
- link link_right_wrist_roll: geometry collision mesh filename=package://x1_urdf/robot/x1_29dof/meshes/right_wrist_roll.STL; visual mesh filename=package://x1_urdf/robot/x1_29dof/meshes/right_wrist_roll.STL
- link x1-body: geometry collision mesh filename=package://x1_urdf/robot/x1_29dof/meshes/base_link_simple.STL; collision mesh filename=package://x1_urdf/robot/x1_29dof/meshes/base_link_simple.STL
Joints:
- added joint base_to_x1_body_joint: type fixed, parent base_link, child x1-body, origin xyz=0 0 0 rpy=0 0 0

Commit message: feat: sync to newest urdf
fix problem order by alphabetically

File: phc/data/assets/robot/zhiyuan_x1/urdf/x1.urdf (robot description, URDF)
Before this commit: robot zhiyuan scene, 31 links, 30 joints
Links:
- removed link link_lleft_knee_pitch
- added link link_left_knee_pitch, mass 1.68649; collision mesh filename=../meshes/left_knee_pitch.STL; visual mesh filename=../meshes/left_knee_pitch.STL
Joints:
- removed joint left_hip_pitch_joint
- added joint mleft_hip_pitch_joint: type revolute, parent x1-body, child link_left_hip_pitch, origin xyz=0.00245 0.092277 -0.012143 rpy=3.170218624440796e-07 -0.7853990876280905 1.570798162810677, axis 0 0 1, limit lower=-3.14 upper=6.28 effort=150.0 velocity=10
- joint left_ankle_pitch_joint: parent link_lleft_knee_pitch -> link_left_knee_pitch
- joint left_knee_pitch_joint: child link_lleft_knee_pitch -> link_left_knee_pitch

File: phc/data/assets/robot/zhiyuan_x1/urdf/x1_ros.urdf (robot description, URDF)
Before this commit: robot zhiyuan scene, 31 links, 30 joints
Links:
- removed link link_lleft_knee_pitch
- added link link_left_knee_pitch, mass 1.68649; collision mesh filename=package://x1_urdf/robot/x1_29dof/meshes/left_knee_pitch.STL; visual mesh filename=package://x1_urdf/robot/x1_29dof/meshes/left_knee_pitch.STL
Joints:
- removed joint left_hip_pitch_joint
- added joint mleft_hip_pitch_joint: type revolute, parent x1-body, child link_left_hip_pitch, origin xyz=0.00245 0.092277 -0.012143 rpy=3.170218624440796e-07 -0.7853990876280905 1.570798162810677, axis 0 0 1, limit lower=-3.14 upper=6.28 effort=150.0 velocity=10
- joint left_ankle_pitch_joint: parent link_lleft_knee_pitch -> link_left_knee_pitch
- joint left_knee_pitch_joint: child link_lleft_knee_pitch -> link_left_knee_pitch
